File: Fascia.kicad_sch (KiCad schematic)
At the start: 1 part, among them J1 Verdin iMX95

Commit message: Wire the power tree: LM74930-Q1 front end and LM61460-Q1 5 V buck
Both regulators are now fully wired, with every pin either netted or
explicitly NoConnected. ERC sits at 51 findings, all expected: the 50 X1
pins awaiting the bridge/transceiver/codec/panel blocks, plus IGN_SENSE,
which has no destination until the ignition-sense path reaches a module
ADC pin.

Front end follows TI's own reference circuit for the part, "VBAT 12-V or
24-V With 200-V Unsuppressed Load Dump - Output Clamp": back-to-back
FETs with A and OUT on the shared source node, the sense resistor with
its 50-ohm tap into CS+, and OVCLAMP tied to OV so the part clamps
through a surge with circuit-breaker timing rather than disconnecting.
That one net is the whole reason the module rides through a load dump
instead of rebooting.

Buck wires BIAS to the output rail (valid only because Vout <= 12 V),
the boot network through RBOOT, FB/EN dividers, RT, and pull-ups on the
open-drain FLT and PGOOD outputs - those two are a real design
requirement, not an ERC workaround; open-drain outputs do nothing
without them.

Infrastructure added: a generic rectangular symbol factory driven off
parts.py, and a declarative pin-name -> net mapping so a part's wiring
reads as a table rather than as coordinate arithmetic. Rails use power
symbols, everything else uses stub-and-label, and the two mechanisms are
kept strictly separate per this project's KiCad notes. Any pin absent
from a part's net map gets a real NoConnect rather than being left
dangling.

Two bugs found and fixed on the way, both of the class ERC either
catches confusingly or cannot catch at all:

- The generic symbol width was snapped to 1.27 rather than 2.54. Since
  pins sit at +/-(width/2 + LEAD), an odd multiple of 1.27 put every pin
  half a grid step off, which broke the assumption place_part's snap()
  depends on. It surfaced not as one tidy error but as a 114-finding
  cascade - off-grid pins, then wires whose ends missed those pins, then
  dang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
Parts:
- added C1: 100uF, symbol Fascia:C
- added C2: 100n CVS, symbol Fascia:C
- added C3: 100n CCAP, symbol Fascia:C
- added C4: open CT, symbol Fascia:C
- added C5: 10u in, symbol Fascia:C
- added C6: 1u VCC, symbol Fascia:C
- added C7: 100n boot, symbol Fascia:C
- added C8: 44u out, symbol Fascia:C
- added D1: TVS 33V, symbol Fascia:TVS
- added F1: 5A, symbol Fascia:FUSE
- added J2: Power in, symbol Fascia:CONN3
- added L1: 2.2u, symbol Fascia:L
- added Q1: NFET diode, symbol Fascia:NFET
- added Q2: NFET pass, symbol Fascia:NFET
- added R1: 2m sense, symbol Fascia:R
- added R10: FB top, symbol Fascia:R
- added R11: FB bot, symbol Fascia:R
- added R12: RT, symbol Fascia:R
- added R13: EN top, symbol Fascia:R
- added R14: EN bot, symbol Fascia:R
- added R15: 100k FLT pu, symbol Fascia:R
- added R16: 100k PG pu, symbol Fascia:R
- added R2: 50R, symbol Fascia:R
- added R3: RILIM, symbol Fascia:R
- added R4: 5k RMON, symbol Fascia:R
- added R5: OV top, symbol Fascia:R
- added R6: OV bot, symbol Fascia:R
- added R7: UV top, symbol Fascia:R
- added R8: UV bot, symbol Fascia:R
- added R9: RBOOT, symbol Fascia:R
- added U1: LM74930-Q1, symbol Fascia:LM74930-Q1
- added U2: LM61460-Q1, symbol Fascia:LM61460-Q1
Connections:
- net +5V: now also C8.1, L1.2, R10.1, R15.2, R16.2, U2.1 (BIAS)
- net GND: now also C1.2, C2.2, C4.2, C5.2, C6.2, C8.2, D1.2, J2.2 (GND), R11.2, R12.2, R14.2, R3.2, R4.2, R6.2, R8.2, U1.13 (GND), U2.11 (PGND2), U2.3 (AGND), U2.9 (PGND1)
- new net +12V_PROT: C5.1, Q1.2 (D), R13.1, U1.18 (ISCP), U1.24 (C), U2.12 (VIN2), U2.8 (VIN1)
- new net BOOT_C: C7.1, R9.2, U2.14 (CBOOT)
- new net BOOT_R: R9.1, U2.13 (RBOOT)
- new net CAP_CP: C3.1, U1.23 (CAP)
- new net COMMON: Q1.3 (S), Q2.3 (S), U1.15 (OUT), U1.2 (A)
- new net CS_PLUS: R2.2, U1.20 (CS+)
- new net DGATE: Q1.1 (G), U1.1 (DGATE)
- new net EN_5V: R13.2, R14.1, U2.7 (EN/SYNC)
- new net FB_5V: R10.2, R11.1, U2.4 (FB)
- new net HGATE: Q2.1 (G), U1.14 (HGATE)
- new net IGN_SENSE: J2.3 (IGN)
- new net ILIM: R3.1, U1.11 (ILIM)
- new net IMON: R4.1, U1.10 (IMON)
- new net OV_DIV: R5.2, R6.1, U1.16 (OVCLAMP), U1.5 (OV)
- new net PG_5V: R16.1, U2.5 (PGOOD)
- new net PWR_FLT: R15.1, U1.12 (FLT)
- new net RT_5V: R12.1, U2.6 (RT)
- new net SENSE_OUT: Q2.2 (D), R1.2, U1.19 (CS-)
- new net SW_5V: C7.2, L1.1, U2.10 (SW)
- new net SW_SENSE: R5.1, R7.1, U1.3 (SW)
- new net TMR: C4.1, U1.9 (TMR)
- new net UVLO_DIV: R7.2, R8.1, U1.4 (UVLO)
- new net VBAT_F: C1.1, C2.1, C3.2, D1.1, F1.2, R1.1, R2.1, U1.22 (VS), U1.6 (EN), U1.7 (MODE)
- new net VBAT_IN: F1.1, J2.1 (VBAT)
- new net VCC_LDO: C6.1, U2.2 (VCC)
- no-connect marks 158 -> 161

Commit message: Wire the 1.8 V rail and the CAN FD link to ecu-pcb
Adds the TLV767-Q1 1.8 V LDO and the TCAN1044V-Q1 CAN transceiver, and
connects the module's CAN_1_TX / CAN_1_RX to them. ERC drops from 51 to
49 findings, still all expected: 48 X1 pins awaiting the bridge, codec
and panel connector, plus IGN_SENSE.

The 1.8 V rail exists because the Verdin's I/O is 1.8 V logic. An LDO
rather than a buck on purpose - the load is small, and a linear
regulator adds no switching noise to a board carrying LVDS next to a car
radio. It feeds the transceiver's VIO now and the SN65DSI85-Q1 bridge
later.

CAN uses split termination - 2x60 ohm with a midpoint capacitor to
ground - rather than a single 120 ohm, because the midpoint cap shunts
common-mode noise on a bus that leaves the enclosure on a harness. STB
gets a pull-down: the part has an internal pull-up, so without it the
transceiver would wake in standby and the link would simply not work.

TLV767-Q1 added to parts.py with two notes. Pin 3 differs between
versions - FB on the adjustable part, SNS on the fixed one - and this
design uses the adjustable version. And its thermal pad MAY be grounded,
which is worth stating explicitly right below the LM74930-Q1 whose pad
must NOT be; neither part's pad rule generalises to the other.

One real bug found by ERC, and it was a good signal rather than noise:
once the LDO was placed, +1V8 had a genuine power_out driving it, so the
PWR_FLAG that had been standing in for a driver became a second power
output on the same net - a pin_to_pin error. The flag logic now tracks
which rails a real part drives and only flags the undriven ones. The
build prints both lists, so "+1V8 and VCC_LDO have real drivers, the
other four are still flagged" is visible on every run rather than
implicit.

Also refreshed two stale README passages left over from the scope
change: the carrier-board summary now mentions audio, USB-C and the
bridge, and notes that Bluetooth and Wi-Fi need no carrier hardware.

Co-Authored-By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
Parts:
- added C10: 10u out, symbol Fascia:C
- added C11: 100n VCC, symbol Fascia:C
- added C12: 100n VIO, symbol Fascia:C
- added C13: 4n7 split, symbol Fascia:C
- added C9: 10u in, symbol Fascia:C
- added J3: CAN to ECU, symbol Fascia:CONN_CAN
- added R17: FB top, symbol Fascia:R
- added R18: FB bot, symbol Fascia:R
- added R19, R20: 60R term, symbol Fascia:R
- added R21: 10k STB pd, symbol Fascia:R
- added U3: TLV767-Q1, symbol Fascia:TLV767-Q1
- added U4: TCAN1044V-Q1, symbol Fascia:TCAN1044V-Q1
Connections:
- net +5V: now also C11.1, C9.1, U3.5 (EN), U3.8 (IN), U4.3 (VCC)
- net GND: now also C10.2, C11.2, C12.2, C13.2, C9.2, J3.3 (GND), R18.2, R21.2, U3.4 (GND), U3.6 (GND2), U4.2 (GND)
- net CAN1_TXD: now reaches J1.20 (CAN_1_TX)
- net CAN1_TXD: now also U4.1 (TXD)
- net CAN1_RXD: now reaches J1.22 (CAN_1_RX)
- net CAN1_RXD: now also U4.4 (RXD)
- new net +1V8: C10.1, C12.1, R17.1, U3.1 (OUT), U4.5 (VIO)
- new net CAN1_H: J3.1 (CANH), R19.1, U4.7 (CANH)
- new net CAN1_L: J3.2 (CANL), R20.2, U4.6 (CANL)
- new net CAN1_SPLIT: C13.1, R19.2, R20.1
- new net CAN1_STB: R21.1, U4.8 (STB)
- new net FB_1V8: R17.2, R18.1, U3.3 (FB)
- no-connect marks 161 -> 163

Commit message: Wire the SN65DSI85-Q1 bridge: the display path is complete end to end
Adds the DSI-to-LVDS bridge and a provisional panel connector, and
connects the module's full DSI link to it. ERC drops from 49 to 37,
still all expected.

The milestone is the display bank: it is down from 15 unconnected pins
to 2. The whole path from the module's MIPI DSI, through the bridge, out
as dual-link LVDS to the panel connector, is wired. The only thing
missing from it is the backlight - PWM_3_DSI and GPIO_10_DSI - which
cannot be designed until iFan send the string voltage and current.

Configured for datasheet Table 5 "Single DSI Input to Dual-Link LVDS":
DSI channel A, four lanes, odd pixels on LVDS link A and even on B.

Five datasheet requirements that are easy to get wrong, all handled and
all recorded in parts.py:

- VCORE (31) is the 1.1 V regulator OUTPUT, not a supply input. It gets
  its 1 uF to ground; feeding it would destroy the part. The build's
  driven-rail tracking picked it up automatically and correctly withheld
  a PWR_FLAG from it.
- The unused DSI channel B inputs must be left UNCONNECTED, not tied
  off. The datasheet says so twice - in the pin table and again under
  CHA_DSI_LANES. They get NoConnect items, visible as X marks on the
  drawing.
- RSVD1 (34) and RSVD2 (1) likewise "must be left unconnected for normal
  operation".
- REFCLK (17) is unused here, since the LVDS pixel clock comes from the
  free-running D-PHY clock - but unused means resistor-pulled to ground,
  not floating.
- ADDR (64) is strapped low for a defined I2C address. Worth noting that
  strapping it HIGH would have required tying it to the same 1.8 V rail
  as VCC, not merely to a 1.8 V rail.

parts.py asserts the part has exactly 64 pins and exactly 12 VCC pins -
a dropped supply pin is a brownout that nothing on the drawing shows.

Also recorded that this part's PowerPAD IS reference ground, in contrast
to the LM74930-Q1's which must float. That is now three parts in one
file with three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
Parts:
- added C14: 1u VCORE, symbol Fascia:C
- added C15: 10u 1V8, symbol Fascia:C
- added C16, C17, C18, C19, C20, C21: 100n 1V8, symbol Fascia:C
- added J4: Panel LVDS (provisional), symbol Fascia:CONN_PANEL
- added R22: 10k REFCLK, symbol Fascia:R
- added U5: SN65DSI85-Q1, symbol Fascia:SN65DSI85-Q1
Connections:
- net +1V8: now also C15.1, C16.1, C17.1, C18.1, C19.1, C20.1, C21.1, U5.14 (VCC2), U5.18 (VCC3), U5.3 (VCC1), U5.32 (VCC4), U5.35 (VCC5), U5.40 (VCC6), U5.43 (VCC7), U5.48 (VCC8), U5.49 (VCC9), U5.55 (VCC10), U5.58 (VCC11), U5.63 (VCC12)
- net GND: now also C14.2, C15.2, C16.2, C17.2, C18.2, C19.2, C20.2, C21.2, J4.21 (GND1), J4.22 (GND2), R22.2, U5.23 (GND1), U5.26 (GND2), U5.52 (GND3), U5.64 (ADDR)
- net DSI_BRIDGE_EN: now reaches J1.17 (GPIO_9_DSI)
- net DSI_BRIDGE_EN: now also U5.2 (EN)
- net DSI_D3_N: now reaches J1.23 (DSI_1_D3_N)
- net DSI_D3_N: now also U5.30 (DA3N)
- net DSI_D3_P: now reaches J1.25 (DSI_1_D3_P)
- net DSI_D3_P: now also U5.29 (DA3P)
- net DSI_D2_N: now reaches J1.29 (DSI_1_D2_N)
- net DSI_D2_N: now also U5.28 (DA2N)
- net DSI_D2_P: now reaches J1.31 (DSI_1_D2_P)
- net DSI_D2_P: now also U5.27 (DA2P)
- net DSI_CLK_N: now reaches J1.35 (DSI_1_CLK_N)
- net DSI_CLK_N: now also U5.25 (DACN)
- net DSI_CLK_P: now reaches J1.37 (DSI_1_CLK_P)
- net DSI_CLK_P: now also U5.24 (DACP)
- net DSI_D1_N: now reaches J1.41 (DSI_1_D1_N)
- net DSI_D1_N: now also U5.22 (DA1N)
- net DSI_D1_P: now reaches J1.43 (DSI_1_D1_P)
- net DSI_D1_P: now also U5.21 (DA1P)
- net DSI_D0_N: now reaches J1.47 (DSI_1_D0_N)
- net DSI_D0_N: now also U5.20 (DA0N)
- net DSI_D0_P: now reaches J1.49 (DSI_1_D0_P)
- net DSI_D0_P: now also U5.19 (DA0P)
- net DSI_I2C_SDA: now reaches J1.53 (I2C_2_DSI_SDA)
- net DSI_I2C_SDA: now also U5.16 (SDA)
- net DSI_I2C_SCL: now reaches J1.55 (I2C_2_DSI_SCL)
- net DSI_I2C_SCL: now also U5.15 (SCL)
- new net DSI_IRQ: U5.33 (IRQ)
- new net LVDS_A_CLKN: J4.10 (A_CLKN), U5.39 (A_CLKN)
- new net LVDS_A_CLKP: J4.9 (A_CLKP), U5.38 (A_CLKP)
- new net LVDS_A_Y0N: J4.2 (A_Y0N), U5.47 (A_Y0N)
- new net LVDS_A_Y0P: J4.1 (A_Y0P), U5.46 (A_Y0P)
- new net LVDS_A_Y1N: J4.4 (A_Y1N), U5.45 (A_Y1N)
- new net LVDS_A_Y1P: J4.3 (A_Y1P), U5.44 (A_Y1P)
- new net LVDS_A_Y2N: J4.6 (A_Y2N), U5.42 (A_Y2N)
- new net LVDS_A_Y2P: J4.5 (A_Y2P), U5.41 (A_Y2P)
- new net LVDS_A_Y3N: J4.8 (A_Y3N), U5.37 (A_Y3N)
- new net LVDS_A_Y3P: J4.7 (A_Y3P), U5.36 (A_Y3P)
- new net LVDS_B_CLKN: J4.20 (B_CLKN), U5.54 (B_CLKN)
- new net LVDS_B_CLKP: J4.19 (B_CLKP), U5.53 (B_CLKP)
- new net LVDS_B_Y0N: J4.12 (B_Y0N), U5.62 (B_Y0N)
- new net LVDS_B_Y0P: J4.11 (B_Y0P), U5.61 (B_Y0P)
- new net LVDS_B_Y1N: J4.14 (B_Y1N), U5.60 (B_Y1N)
- new net LVDS_B_Y1P: J4.13 (B_Y1P), U5.59 (B_Y1P)
- new net LVDS_B_Y2N: J4.16 (B_Y2N), U5.57 (B_Y2N)
- new net LVDS_B_Y2P: J4.15 (B_Y2P), U5.56 (B_Y2P)
- new net LVDS_B_Y3N: J4.18 (B_Y3N), U5.51 (B_Y3N)
- new net LVDS_B_Y3P: J4.17 (B_Y3P), U5.50 (B_Y3P)
- new net REFCLK_GND: R22.1, U5.17 (REFCLK)
- new net VCORE_1V1: C14.1, U5.31 (VCORE)
- no-connect marks 163 -> 175

Commit message: Wire the audio block; catch a codec/module logic-level incompatibility
Adds the PCM3168A-Q1 codec, a 3.3 V rail, two SN74AXC4T245-Q1 level
shifters and the pre-out and microphone connectors. ERC 37 -> 35, and
bank D is down to just USB-C and the second CAN.

The finding that shaped this block: the codec's digital domain is
3.0-3.6 V and cannot be run at 1.8 V. Its VIH minimum is 2 V, above what
a 1.8 V output can guarantee - and its VOH minimum is 2.4 V, above the
module's 2.1 V ABSOLUTE MAXIMUM on 1.8 V I/O. Wired directly, the
codec-to-module direction would have damaged the module. Every digital
line between them is now translated.

I2S and clocks go through SN74AXC4T245-Q1 (AEC-Q100, 0.65-3.6 V per
rail, two independent direction controls, 380 Mbps at 1.8->3.3 V). I2C
uses the classic two-N-FET open-drain translator instead, since a
push-pull part cannot pass a bus where either end may pull low.

Audio: five differential pre-outs (front L/R, rear L/R, sub) on J5, a
microphone into the first differential ADC input biased on the codec's
own VCOMAD reference, TDM on DIN1 so DIN2-4 are unused, and MODE
strapped low to select the I2C control port. The 3.3 V rail reuses the
TLV767-Q1 already chosen for 1.8 V with a different divider - no new BOM
line.

Three bugs found and fixed, in increasing order of severity:

- Bidirectional pins strapped straight to GND drew pin_to_pin errors.
  ERC was right: a bidirectional pin hard-wired to a supply is a short
  the moment anything drives it. They are now tied off through
  resistors, which is better practice regardless.

- Two nets SILENTLY MERGED. The audio block wrapped into more columns
  than its band allowed, and a decoupling cap's ground stub landed
  exactly on the power tree's UVLO_DIV label. ERC does report this
  (multiple_net_names) but only for the pair it happens to notice, so
  build_schematic.py now checks every terminated point directly and
  fails loudly, naming the offending part. The sheet grew A1 -> A0 and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
Parts:
- added C22: 10u in, symbol Fascia:C
- added C23: 10u out, symbol Fascia:C
- added C24: 100n U7A, symbol Fascia:C
- added C25: 100n U7B, symbol Fascia:C
- added C26: 100n U8A, symbol Fascia:C
- added C27: 100n U8B, symbol Fascia:C
- added C28, C29, C30: 10u decouple, symbol Fascia:C
- added C31, C32, C33, C34: 100n codec, symbol Fascia:C
- added C35: 100n RST, symbol Fascia:C
- added C36: 1u couple, symbol Fascia:C
- added J5: Pre-outs to amp, symbol Fascia:CONN_PREOUT
- added J6: Mic, symbol Fascia:CONN_MIC
- added Q3, Q4: NFET i2c xlat, symbol Fascia:NFET
- added R23: FB top, symbol Fascia:R
- added R24: FB bot, symbol Fascia:R
- added R25, R26, R27, R28: 2k2 pullup, symbol Fascia:R
- added R29: 100k RST, symbol Fascia:R
- added R30: 2k2 mic bias, symbol Fascia:R
- added R31, R32: 10k bias, symbol Fascia:R
- added R33, R34, R35, R36: 10k tie-off, symbol Fascia:R
- added U6: TLV767-Q1 3V3, symbol Fascia:TLV767-Q1
- added U7, U8: SN74AXC4T245-Q1, symbol Fascia:SN74AXC4T245-Q1
- added U9: PCM3168A-Q1, symbol Fascia:PCM3168A-Q1
Connections:
- net +1V8: now also C24.1, C26.1, Q3.1 (G), Q4.1 (G), R25.2, R26.2, U7.1 (VCCA), U7.2 (1DIR), U7.3 (2DIR), U8.1 (VCCA), U8.3 (2DIR)
- net +5V: now also C22.1, C31.1, C32.1, R30.1, U6.5 (EN), U6.8 (IN), U9.14 (VCCDA1), U9.3 (VCCAD2), U9.34 (VCCDA2), U9.49 (VCCAD1)
- net GND: now also C22.2, C23.2, C24.2, C25.2, C26.2, C27.2, C28.2, C29.2, C30.2, C31.2, C32.2, C33.2, C34.2, C35.2, J5.11 (GND), J6.3 (GND), R24.2, R33.2, R34.2, R35.2, R36.2, U6.4 (GND), U6.6 (GND2), U7.14 (2OE), U7.15 (1OE), U7.8 (GND1), U7.9 (GND2), U8.14 (2OE), U8.15 (1OE), U8.2 (1DIR), U8.8 (GND1), U8.9 (GND2), U9.11 (DGND2), U9.16 (AGNDDA1), U9.2 (AGNDAD2), U9.33 (AGNDDA2), U9.45 (ADR0), U9.47 (DGND1), U9.48 (MODE), U9.50 (AGNDAD1), U9.60 (VREFAD2)
- net I2C1_SDA_1V8: now reaches J1.12 (I2C_1_SDA)
- net I2C1_SDA_1V8: now also Q3.3 (S), R25.1
- net I2C1_SCL_1V8: now reaches J1.14 (I2C_1_SCL)
- net I2C1_SCL_1V8: now also Q4.3 (S), R26.1
- new net +3V3: C23.1, C25.1, C27.1, C33.1, C34.1, R23.1, R27.2, R28.2, R29.1, U6.1 (OUT), U7.16 (VCCB), U8.16 (VCCB), U9.12 (VDD2), U9.46 (VDD1)
- new net AOUT_FL_N: J5.2 (FL_N), U9.32 (VOUT1N)
- new net AOUT_FL_P: J5.1 (FL_P), U9.31 (VOUT1P)
- new net AOUT_FR_N: J5.4 (FR_N), U9.30 (VOUT2N)
- new net AOUT_FR_P: J5.3 (FR_P), U9.29 (VOUT2P)
- new net AOUT_RL_N: J5.6 (RL_N), U9.28 (VOUT3N)
- new net AOUT_RL_P: J5.5 (RL_P), U9.27 (VOUT3P)
- new net AOUT_RR_N: J5.8 (RR_N), U9.26 (VOUT4N)
- new net AOUT_RR_P: J5.7 (RR_P), U9.25 (VOUT4P)
- new net AOUT_SUB_N: J5.10 (SUB_N), U9.24 (VOUT5N)
- new net AOUT_SUB_P: J5.9 (SUB_P), U9.23 (VOUT5P)
- new net CODEC_DOUT_1V8: J1.36 (I2S_1_D_IN), U8.4 (1A1)
- new net CODEC_DOUT_3V3: U8.13 (1B1), U9.8 (DOUT1)
- new net CODEC_RST: C35.1, R29.2, U9.4 (RST)
- new net CODEC_SCL_3V3: Q4.2 (D), R28.1, U9.42 (SCL)
- new net CODEC_SDA_3V3: Q3.2 (D), R27.1, U9.43 (SDA)
- new net FB_3V3: R23.2, R24.1, U6.3 (FB)
- new net I2S_BCK_1V8: J1.30 (I2S_1_BCLK), U7.4 (1A1)
- new net I2S_BCK_3V3: U7.13 (1B1), U9.36 (BCKDA), U9.7 (BCKAD)
- new net I2S_DIN_1V8: J1.34 (I2S_1_D_OUT), U7.6 (2A1)
- new net I2S_DIN_3V3: U7.11 (2B1), U9.37 (DIN1)
- new net I2S_LRCK_1V8: J1.32 (I2S_1_SYNC), U7.5 (1A2)
- new net I2S_LRCK_3V3: U7.12 (1B2), U9.35 (LRCKDA), U9.6 (LRCKAD)
- new net I2S_SCKI_1V8: J1.38 (I2S_1_MCLK), U7.7 (2A2)
- new net I2S_SCKI_3V3: U7.10 (2B2), U9.41 (SCKI)
- new net MIC_BIAS_P: C36.1, J6.1 (MIC_P), R30.2
- new net MIC_IN_N: J6.2 (MIC_N), R32.2, U9.51 (VIN1N)
- new net MIC_IN_P: C36.2, R31.2, U9.52 (VIN1P)
- new net U8_1B2_TIE: R33.1, U8.12 (1B2)
- new net U8_2A1_TIE: R34.1, U8.6 (2A1)
- new net U8_2A2_TIE: R35.1, U8.7 (2A2)
- new net U9_ADR1_TIE: R36.1, U9.44 (ADR1)
- new net VCOMAD: C28.1, R31.1, R32.1, U9.1 (VCOMAD)
- new net VCOMDA: C29.1, U9.15 (VCOMDA)
- new net VREFAD1: C30.1, U9.59 (VREFAD1)
- no-connect marks 175 -> 198
