File: Fascia.kicad_sch (KiCad schematic)
At the start: 118 parts, among them J1 Verdin iMX95, J10 RTC coin cell, J2 Power in, J3 CAN to ECU, J4 Panel LVDS (provisional), J5 Pre-outs to amp, J6 Mic, J7 USB-C CarPlay, J8 JTAG debug, J9 Buttons, Q1 NFET diode, Q2 NFET pass, Q3 NFET i2c xlat, Q4 NFET i2c xlat, U1 LM74930-Q1, U10 TPS2557-Q1, U2 LM61460-Q1, U3 TLV767-Q1, U4 TCAN1044V-Q1, U5 SN65DSI85-Q1, U6 TLV767-Q1 3V3, U7 SN74AXC4T245-Q1, U8 SN74AXC4T245-Q1, U9 PCM3168A-Q1

Commit message: Assign and verify footprints; make exposed-pad handling explicit
Every part except one now carries a KiCad library footprint, and
build_schematic.py verifies at build time that each named file actually
exists. A mistyped library path is otherwise invisible until the netlist
reaches the PCB editor and silently drops the part.

The biggest footprint risk turned out to be none at all: the Verdin
plugs into a standard DDR4 SODIMM socket, and KiCad's
SODIMM-260_DDR4_H4.0-5.2_OrientationStd_Socket has exactly 260 pads
numbered 1-260 - a direct match for the extracted pinout, checked rather
than assumed.

The one gap is the LM61460-Q1. Its RJR (VQFN-HR-14) package has no
KiCad footprint and needs generating, the way the sibling projects
generate their odd packages. The build prints it as outstanding on every
run rather than leaving it to be noticed later.

Exposed pads needed real thought. All of these footprints number the pad
N+1 - 65 on the TQFP-64s, 25 on the VQFN-24, 9 on the SON-8s - so each
symbol now carries an explicit EP pin and the schematic states what
happens to it:

  LM74930-Q1                  NoConnect; the datasheet forbids grounding
  TLV767-Q1, TPS2557-Q1       GND
  SN65DSI85-Q1, PCM3168A-Q1   GND (PowerPAD is reference ground)

The LM74930-Q1's NoConnect is the load-bearing one. Without an explicit
pin that pad would merely be netless, and nothing on the drawing would
stop a later ground-stitching pass from claiming it - which is exactly
how that part gets destroyed. Three parts in this design have three
different pad rules; none generalises to the others.

ERC unchanged at 10, all still blocked or optional.

Co-Authored-By: Claude Opus 5 <noreply@anthropic.com>
Parts:
- C1, C10, C11, C12, C13, C14, C15, C16, C17, C18, C19, C2, C20, C21, C22, C23, C24, C25, C26, C27, C28, C29, C3, C30, C31, C32, C33, C34, C35, C36, C37, C38, C39, C4, C5, C6, C7, C8, C9: footprint (none) -> Capacitor_SMD:C_0603_1608Metric
- D1, D2, D3, D4: footprint (none) -> Diode_SMD:D_SMB
- F1: footprint (none) -> Fuse:Fuse_Bourns_MF-RG300
- J1: footprint (none) -> Connector_PCBEdge:SODIMM-260_DDR4_H4.0-5.2_OrientationStd_Socket
- L1: footprint (none) -> Inductor_SMD:L_1210_3225Metric
- Q1, Q2, Q3, Q4: footprint (none) -> Package_TO_SOT_SMD:SOT-23
- R1, R10, R11, R12, R13, R14, R15, R16, R17, R18, R19, R2, R20, R21, R22, R23, R24, R25, R26, R27, R28, R29, R3, R30, R31, R32, R33, R34, R35, R36, R37, R38, R39, R4, R40, R41, R42, R43, R44, R45, R46, R47, R48, R49, R5, R6, R7, R8, R9: footprint (none) -> Resistor_SMD:R_0603_1608Metric
- U1: footprint (none) -> Package_DFN_QFN:Texas_RGE0024H_VQFN-24-1EP_4x4mm_P0.5mm_EP2.7x2.7mm
- U10, U3, U6: footprint (none) -> Package_DFN_QFN:Texas_DRB0008A
- U4: footprint (none) -> Package_SO:SOIC-8_3.9x4.9mm_P1.27mm
- U5, U9: footprint (none) -> Package_QFP:Texas_TQFP-64-1EP_10x10mm_P0.5mm_EP8x8mm_Mask4.44x4.44mm
- U7, U8: footprint (none) -> Package_SO:TSSOP-16_4.4x5mm_P0.65mm
Connections:
- net GND: now also U10.9 (EP), U3.9 (EP), U5.65 (EP), U6.9 (EP), U9.65 (EP)
- no-connect marks 207 -> 208

Commit message: Generate the LM61460-Q1 VQFN-HR-14 footprint; every part now has one
TI's RJR0014A has no KiCad library footprint and is not something a
generic QFN generator can produce: the pads are all different sizes,
unevenly spaced, and the four corner pads are L-shaped. This was the last
thing blocking the PCB.

Geometry is not eyeballed off the drawing. The LAND PATTERN EXAMPLE on
page 55 of TI SNVSB70F is real vector art, so the pad rectangles were
extracted from the PDF's own path data with PyMuPDF and only the scale
had to be inferred - from a dimension the drawing states outright, pad 10
being 2.4 x 0.4 mm. That scale then reproduced pad 10's 0.400 mm height
exactly, which is what makes the rest of the extraction trustworthy.

Each L-shaped pad is two rectangles sharing one pad number. That is a
real KiCad construction this project has met before - the Keystone fuse
holder with two physical pads both numbered "1" - and it is far safer
than approximating an L with its bounding box, which would put copper in
the notch and eat the clearance to its neighbours.

All four notches face the outer corner of the pattern. I confirmed that
by rendering the drawing around pads 1, 9 and 11 rather than assuming the
symmetry held, having already been caught once this session assuming a
mirror.

The generator verifies itself twice. Internally: pin numbering, which
pads are L-shaped, pad 10's dimensions, the overall 4.40 x 3.90 extent,
and that no two DIFFERENT pins overlap (same-pin rectangles are supposed
to). Then by loading the result back through KiCad's own pcbnew, which
reports 18 pads, numbers 1-14 with four doubled, and the extent.

That second check earned its place immediately. The first version emitted
trailing "; PINNAME" comments on the pad lines - KiCad's s-expression
format has no comment syntax at all, and the entire library failed to
load with nothing more useful than "Unable to load library". Internal
consistency cannot tell you whether KiCad will accept the file.

Lib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
Parts:
- U2: footprint (none) -> TI_RJR0014A_VQFN-HR:TI_RJR0014A_VQFN-HR-14_4x3.5mm

Commit message: Start the PCB: 118 parts placed and netted, schematic parity clean
Adds build_pcb.py and run_drc.py. The board now exists: 118 footprints,
574 pads netted across 129 nets, six layers, 148 x 164 mm. Nothing is
routed - route_board.py is next.

Ground truth comes from outside this script, deliberately. The parts list
is read out of the schematic file and the net assignments come from
kicad-cli's own netlist export, so drift between schematic and PCB fails
here rather than producing a quietly wrong board. That check is already
earning its keep: DRC reports schematic parity 0.

Six layers rather than four - the DSI and LVDS pairs each want a
reference plane beside them, and the audio section wants a quiet return
of its own.

Connector footprints are PROVISIONAL 2.54 mm headers so the board can be
placed and routed end to end. Every one is a real decision still to make,
and two are blocked: the panel connector waits on the iFan datasheet (the
real part is a 60-pin FFC, not a 22-pin header) and USB-C needs a 24-pad
receptacle with a matching 24-pin symbol.

Three real problems found and fixed on the way:

- TI's DRB0008A footprint carries 0.2 mm thermal vias inside its exposed
  pad, below KiCad's default 0.3 mm minimum hole - 12 drill_out_of_range
  violations. Those vias are how a regulator's heat reaches the inner
  planes, so the board constraint is relaxed to 0.2 mm deliberately
  rather than the footprint being swapped for one without them.

- The board outline was drawn around a PREDICTED size. The packer works
  in bounding boxes, so if any bbox understates a footprint the
  prediction is quietly wrong and parts sit outside the board edge -
  which DRC does not report, because an unrouted board has no copper
  crossing the edge yet. The outline is now measured from where the parts
  actually ended up, and a check asserts all 118 are inside it.

- Chased lib_footprint_mismatch down properly rather than muting it.
  Seven of the eight affected footprints are OLD-FOR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
Parts:
- J10: footprint (none) -> Battery:BatteryHolder_Keystone_1058_1x2032
- J2, J3, J6: footprint (none) -> Connector_PinHeader_2.54mm:PinHeader_1x03_P2.54mm_Vertical
- J4: footprint (none) -> Connector_PinHeader_2.54mm:PinHeader_1x22_P2.54mm_Vertical
- J5: footprint (none) -> Connector_PinHeader_2.54mm:PinHeader_1x11_P2.54mm_Vertical
- J7: footprint (none) -> Connector_PinHeader_2.54mm:PinHeader_1x09_P2.54mm_Vertical
- J8: footprint (none) -> Connector_PinHeader_2.54mm:PinHeader_1x08_P2.54mm_Vertical
- J9: footprint (none) -> Connector_PinHeader_2.54mm:PinHeader_1x04_P2.54mm_Vertical
